File: hardware/pilot/pilot.sch (EAGLE design)
At the start: 23 parts, among them IC1 74HC595N, J1 AVR_SPI_PROG_3X2NS

Commit message: fix sch hc595 wiring
Connections:
- removed net RCK: IC1A.RCK
- net D10: now also IC1A.RCK; no longer IC1A.SCL
- net VCC: now also IC1A.SCL
